Commit message: Use meaningful inertial parameter

File: gz_ros2_control_demos/urdf/test_ackermann_drive.xacro.urdf (robot description, URDF)
Before this commit: robot ackermann_drive, 8 links, 7 joints
Links:
- link chassis: mass 1 -> 100
- link front_left_wheel: mass 2 -> 11.3
- link front_right_wheel: mass 2 -> 11.3
- link rear_left_wheel: mass 2 -> 11.3
- link rear_right_wheel: mass 2 -> 11.3

Commit message: Configure steering joints properly

File: gz_ros2_control_demos/urdf/test_ackermann_drive.xacro.urdf (robot description, URDF)
Before this commit: robot ackermann_drive, 8 links, 7 joints
Joints:
- joint left_wheel_steering_joint: limit (none) -> lower=-1.57 upper=1.57 effort=1000.0 velocity=30; origin xyz=0.9 0.5 -0.2 rpy=-1.57 0 0 -> xyz=0.9 -0.5 -0.2 rpy=1.57 0 0; type continuous -> revolute
- joint right_wheel_steering_joint: limit (none) -> lower=-1.57 upper=1.57 effort=1000.0 velocity=30; origin xyz=0.9 -0.5 -0.2 rpy=-1.57 0 0 -> xyz=0.9 0.5 -0.2 rpy=1.57 0 0; type continuous -> revolute
